Commit message: newrobot

File: robot.urdf (robot description, URDF)
Before this commit: robot my_robot, 14 links, 13 joints
Joints:
- joint joint_1: limit lower=-1.64104 upper=1.50055 effort=10 velocity=10 -> lower=-1.5708 upper=1.5708 effort=10 velocity=10
- joint joint_2: limit lower=-0.215989 upper=1.87841 effort=10 velocity=10 -> lower=-1.5708 upper=0.523599 effort=10 velocity=10; origin xyz=-0.0017197 0.02444 -0.0458276 rpy=1.5708 0 0.0702486 -> xyz=-1.0941e-08 0.0245004 -0.0458276 rpy=1.5708 0 4.46576e-07
- joint joint_3: limit lower=-1.70606 upper=0.388333 effort=10 velocity=10 -> lower=-0.523599 upper=1.5708 effort=10 velocity=10; origin xyz=0.0326611 -0.148961 0.005544 rpy=-0 -0 -0.172343 -> xyz=0.1525 -2.23277e-05 0.005544 rpy=-0 0 0
- joint joint_4: limit lower=-1.73961 upper=0.354782 effort=10 velocity=10 -> lower=-0.523599 upper=1.5708 effort=10 velocity=10; origin xyz=0.1235 0 -0 rpy=0 -0 0 -> xyz=0.1235 0 -0 rpy=-0 0 0
- joint joint_5: limit lower=-1.59462 upper=1.54698 effort=10 velocity=10 -> lower=-1.5708 upper=1.5708 effort=10 velocity=10; origin xyz=0.029387 0.0548578 0.01895 rpy=-1.5708 -0 2.78681 -> xyz=0.06165 -0.0085 0.01895 rpy=-1.5708 -0 1.5708
- joint joint_6: limit lower=-0.488858 upper=0.907405 effort=10 velocity=10 -> lower=-1.0472 upper=0.349066 effort=10 velocity=10; origin xyz=0.00349633 0.0190887 -0.03 rpy=1.5708 -0.663391 1.59462 -> xyz=0.00395 0.019 -0.03 rpy=1.5708 -1.22173 1.5708
- joint joint_6_mimic_L1: origin xyz=0.00365115 0.0125905 -0.0551744 rpy=1.5708 -0 1.59462 -> xyz=0.00395 0.0125 -0.0551744 rpy=1.5708 0 1.5708
- joint joint_6_mimic_L2: origin xyz=-0.0206236 0.0158325 0 rpy=3.14159 -0 3.14159 -> xyz=-0.0258793 0.00250215 0 rpy=-3.14159 -0 3.14159
- joint joint_6_mimic_L3: origin xyz=0.0307896 -0.0393954 -0 rpy=3.14159 -0 -2.4782 -> xyz=0.0469846 -0.017101 0 rpy=-3.14159 0 -1.91986
- joint joint_6_mimic_R1: origin xyz=-0.00365115 -0.0125905 -0.0551744 rpy=-1.5708 -0 1.59462 -> xyz=-0.00395 -0.0125 -0.0551744 rpy=-1.5708 0 1.5708
- joint joint_6_mimic_R2: origin xyz=0.0065 -0.0251744 0 rpy=3.14159 -0 2.4782 -> xyz=0.0065 -0.0251744 0 rpy=3.14159 0 1.91986
- joint joint_6_mimic_R3: origin xyz=-0.0307896 0.0393954 -0 rpy=3.14159 0 3.14159 -> xyz=-0.0469846 0.017101 0 rpy=-3.14159 -0 -3.14159
- joint joint_6_mimic_gear: origin xyz=-0.00349633 -0.0190887 -0.03 rpy=-1.5708 -0 1.59462 -> xyz=-0.00395 -0.019 -0.03 rpy=-1.5708 0 1.5708
