Commit message: globalMin

File: ikpy_robot.urdf (robot description, URDF)
Before this commit: robot my_clean_robot, 7 links, 6 joints
Joints:
- joint joint_1: limit lower=-3.14 upper=3.14 -> lower=-1.57 upper=1.57
- joint tcp_joint: origin xyz=-0.12 0 0 rpy=0 0 0 -> xyz=-0.13 0 0 rpy=0 0 0

Commit message: 최종도착지점 수정

File: ikpy_robot.urdf (robot description, URDF)
Before this commit: robot my_clean_robot, 7 links, 6 joints
Joints:
- joint tcp_joint: origin xyz=-0.12 0 0 rpy=0 0 0 -> xyz=-0.133 0 0 rpy=0 0 0
